File: pcb/IGBS-Rocket-v2_PCB_rev1/IGBS-Rocket-v2_rev1.brd (EAGLE design)
At the start: 151.1 x 34.9 mm, 270 parts, among them IC1 NCV21872DR2G, IC2 NCV21872DR2G, IC3 NCV21872DR2G, J1 U.FL, Q1 BC817, Q2 ENC-03, Q3 BSS316N, Q4 BC817, Q5 BSS314PE, U1 STM32H750VBT6, U10 24AA32A-I/ST, U11 u-blox NEO-M6, U2 LM317BD2TG, U3 CS5171EDR8G, U4 MPU-9250, U5 MICROSD, U6 ESP-12E/F, U7 BMP280, U8 LP324DRG4, U9 MCP6V51T-E/MS, Y1 24MHz

Commit message: * PCB layout fixes
Parts:
- moved TP16 1.02 mm to (71.9, 22.6)
- moved TP10 0.76 mm to (71.9, 28.4)
- moved TP11 0.76 mm to (71.9, 24.6)
- moved TP17 0.76 mm to (71.9, 26.7)
Routing:
- net I2C-AUX-SCL: track 0.00 -> 97.0 mm, vias 0 -> 2
- net I2C-AUX-SDA: track 0.00 -> 94.7 mm, vias 0 -> 2
- net LED4-WHITE: track 0.00 -> 13.9 mm
- net LED2-YELLOW: track 0.00 -> 13.8 mm
- net ESP-IO0: track 56.9 -> 59.5 mm
- net BMP-CS: track 30.6 -> 29.7 mm
- net BMP-MISO: track 34.2 -> 33.4 mm
- net BUZZER: track 53.3 -> 52.6 mm
- net SD-MISO: track 43.4 -> 44.0 mm

Commit message: + PCB layout is complete -> GERBERS are ready
Parts:
- removed U$1: SHORT, testpad2:SHORT
- moved R20 0.25 mm to (69.7, 11.0)
- moved R25 0.25 mm to (69.7, 18.8)
- flipped TP1 to the bottom
Connections:
- net AGND: no longer C20.1, C25.1, C27.2, C29.1, C3.1, C30.1, C34.1, C35.1, C37.1, C38.1, C39.1, C40.1, C41.1, C42.1, C43.1, C8.1, CR2.2, CR2.3, CR3.2, CR3.3, CR4.2, CR4.3, D15.A, IC1.4, IC2.4, IC3.4, Q2.2, R4.3, R6.2, R62.2, R68.3, R70.2, R71.2, R77.3, R79.2, R80.2, U$1.AGND, U3.6, U8.11, U9.4
- net GND: now also C20.1, C25.1, C27.2, C29.1, C3.1, C30.1, C34.1, C35.1, C37.1, C38.1, C39.1, C40.1, C41.1, C42.1, C43.1, C8.1, CR2.2, CR2.3, CR3.2, CR3.3, CR4.2, CR4.3, D15.A, IC1.4, IC2.4, IC3.4, Q2.2, R4.3, R6.2, R62.2, R68.3, R70.2, R71.2, R77.3, R79.2, R80.2, U3.6, U8.11, U9.4; no longer U$1.GND
Routing:
- net 3V3: track 6.96 -> 431.1 mm, vias 0 -> 38
- net 5V: track 0.00 -> 304.4 mm, vias 0 -> 20
- net BAT: track 0.00 -> 105.8 mm
- net 6V: track 0.00 -> 102.7 mm, vias 0 -> 1
- net GND: track 0.00 -> 50.7 mm, vias 0 -> 119
- net 3V3-ESP: track 0.00 -> 30.6 mm, vias 0 -> 4
- net 12V: track 0.00 -> 21.3 mm, vias 0 -> 1
- net GPS-VBCKP: track 0.00 -> 21.2 mm, vias 0 -> 2
- net BAT2: track 0.00 -> 18.0 mm
- net GPS-VCC: track 0.00 -> 17.9 mm, vias 0 -> 3
- net LED2-YELLOW: track 13.8 -> 31.1 mm, vias 0 -> 4
- net VDDA: track 0.00 -> 13.6 mm, vias 0 -> 4
- net 3V3-SD: track 0.00 -> 12.0 mm, vias 0 -> 2
- net 12V-HOT: track 0.00 -> 11.5 mm
- net LED4-WHITE: track 13.9 -> 24.4 mm, vias 0 -> 2
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- added copper zone on layer 1, net GND
- added copper zone on layer 15, net GND
Other:
- board text added: "rev1 18-04-22 JP."
- board text removed: "rev1 23-03-22 JP."
