File: pcb/IGBS-Rocket-v2_PCB_rev1/IGBS-Rocket-v2_rev1.sch (EAGLE design)
At the start: 270 parts, among them IC1 NCV21872DR2G, IC2 NCV21872DR2G, IC3 NCV21872DR2G, J1 U.FL, Q1 BC817, Q2 ENC-03, Q3 BSS316N, Q4 BC817, Q5 BSS314PE, U1 STM32H750VBT6, U10 24AA32A-I/ST, U11 u-blox NEO-M6, U2 LM317BD2TG, U3 CS5171EDR8G, U4 MPU-9250, U5 MICROSD, U6 ESP-12E/F, U7 BMP280, U8 LP324DRG4, U9 MCP6V51T-E/MS, Y1 24MHz

Commit message: + PCB layout is complete -> GERBERS are ready
Parts:
- removed U$1: SHORT, testpad2:SHORT
Connections:
- net AGND: no longer C20.1, C25.1, C27.2, C29.1, C3.1, C30.1, C34.1, C35.1, C37.1, C38.1, C39.1, C40.1, C41.1, C42.1, C43.1, C8.1, CR2.2, CR2.3, CR3.2, CR3.3, CR4.2, CR4.3, D15.A, IC1P.V-, IC2P.V-, IC3P.V-, Q2.GND, R4.3, R6.2, R62.2, R68.3, R70.2, R71.2, R77.3, R79.2, R80.2, U$1.1, U3.AGND, U8P.GND, U9P.GND
- net GND: now also C20.1, C25.1, C27.2, C29.1, C3.1, C30.1, C34.1, C35.1, C37.1, C38.1, C39.1, C40.1, C41.1, C42.1, C43.1, C8.1, CR2.2, CR2.3, CR3.2, CR3.3, CR4.2, CR4.3, D15.A, IC1P.V-, IC2P.V-, IC3P.V-, Q2.GND, R4.3, R6.2, R62.2, R68.3, R70.2, R71.2, R77.3, R79.2, R80.2, U3.AGND, U8P.GND, U9P.GND; no longer U$1.2
